File: C64 Modulator.sch (KiCad schematic (older format))
At the start: 40 parts, among them J10 , J11 , J12 , J13 , J14 , J2 8765, J3 4321, J4 AUD_RIGHT, J5 TRS_3.5mm, J6 RCA_PLUG, J7 , J8 , J9 , Q1 BC549, Q2 BC549, U1 LM7805

Commit message: Cleaned up library for new KiCad & started splitting Chroma/Luma/Comp
Parts:
- removed L1: 22uH, Inductors_THT:L_Axial_L6.6mm_D2.7mm_P10.16mm_Horizontal_Vishay_IM-2, symbol L_Small
- added Q2, Q3: BC549, Package_TO_SOT_THT:TO-92_Inline, symbol Transistor_BJT:BC549
- added R10: 220, Resistor_THT:R_Axial_DIN0207_L6.3mm_D2.5mm_P10.16mm_Horizontal, symbol Device:R
- added R8: 68, Resistor_THT:R_Axial_DIN0207_L6.3mm_D2.5mm_P10.16mm_Horizontal, symbol Device:R
- C3, C6: footprint Capacitors_THT:C_Disc_D4.7mm_W2.5mm_P5.00mm -> Capacitor_THT:C_Disc_D4.7mm_W2.5mm_P5.00mm; symbol C_Small -> Device:C_Small
- C4: renamed from C1; footprint Capacitors_THT:C_Disc_D4.7mm_W2.5mm_P5.00mm -> Capacitor_THT:C_Disc_D4.7mm_W2.5mm_P5.00mm; symbol C_Small -> Device:C_Small
- C5: renamed from C2; footprint Capacitors_THT:C_Disc_D4.7mm_W2.5mm_P5.00mm -> Capacitor_THT:C_Disc_D4.7mm_W2.5mm_P5.00mm; symbol C_Small -> Device:C_Small
- C7: renamed from C4; footprint Capacitors_THT:CP_Radial_D5.0mm_P2.50mm -> Capacitor_THT:CP_Radial_D5.0mm_P2.50mm; symbol CP_Small -> Device:CP_Small
- C8: renamed from C5; footprint Capacitors_THT:CP_Radial_D5.0mm_P2.50mm -> Capacitor_THT:CP_Radial_D5.0mm_P2.50mm; symbol CP1_Small -> Device:CP1_Small
- C9: renamed from C7; footprint Capacitors_THT:C_Disc_D4.7mm_W2.5mm_P5.00mm -> Capacitor_THT:C_Disc_D4.7mm_W2.5mm_P5.00mm; symbol C_Small -> Device:C_Small
- D2: footprint Diodes_THT:D_DO-35_SOD27_P7.62mm_Horizontal -> Diode_THT:D_DO-35_SOD27_P7.62mm_Horizontal; symbol D_Small -> Device:D_Small
- D5: renamed from D1; symbol D_Small -> Device:D_Small
- J1: renamed from J7; symbol Conn_01x01 -> C64-Modulator-rescue:Conn_01x01
- J10: renamed from J3; symbol 6569_4321 -> 6569_modulator:6569_4321
- J11: renamed from J4; symbol Conn_01x02 -> C64-Modulator-rescue:Conn_01x02
- J12: renamed from J5; symbol TRS_3.5mm -> trs_3.5mm:TRS_3.5mm
- J13: renamed from J6; symbol RCA_PLUG -> rca_plug:RCA_PLUG
- J2: renamed from J8; symbol Conn_01x01 -> C64-Modulator-rescue:Conn_01x01
- J3: renamed from J9; symbol Conn_01x01 -> C64-Modulator-rescue:Conn_01x01
- J4: renamed from J10; symbol Conn_01x01 -> C64-Modulator-rescue:Conn_01x01
- J5: renamed from J11; symbol Conn_01x01 -> C64-Modulator-rescue:Conn_01x01
- J6: renamed from J12; symbol Conn_01x01 -> C64-Modulator-rescue:Conn_01x01
- J7: renamed from J13; symbol Conn_01x01 -> C64-Modulator-rescue:Conn_01x01
- J8: renamed from J14; symbol Conn_01x01 -> C64-Modulator-rescue:Conn_01x01
- J9: renamed from J2; symbol 6569_8765 -> 6569_modulator:6569_8765
- JP1: renamed from JP3; footprint Pin_Headers:Pin_Header_Straight_1x02_Pitch2.54mm -> Connector_PinHeader_2.54mm:PinHeader_1x02_P2.54mm_Vertical; symbol Jumper_NC_Small -> Device:Jumper_NC_Small
- JP2: renamed from JP4; footprint Pin_Headers:Pin_Header_Straight_1x02_Pitch2.54mm -> Connector_PinHeader_2.54mm:PinHeader_1x02_P2.54mm_Vertical; symbol Jumper_NC_Small -> Device:Jumper_NC_Small
- JP3: renamed from JP2; symbol Jumper_NC_Dual -> Device:Jumper_NC_Dual
- L1: renamed from L2; footprint Inductors_THT:L_Axial_L6.6mm_D2.7mm_P10.16mm_Horizontal_Vishay_IM-2 -> Inductor_THT:L_Axial_L6.6mm_D2.7mm_P10.16mm_Horizontal_Vishay_IM-2; symbol L_Small -> Device:L_Small
- Q1: renamed from Q2; footprint TO_SOT_Packages_THT:TO-92_Inline_Wide -> Package_TO_SOT_THT:TO-92_Inline; symbol BC549 -> Transistor_BJT:BC549
- Q4: renamed from Q1; footprint TO_SOT_Packages_THT:TO-92_Inline_Wide -> Package_TO_SOT_THT:TO-92_Inline; symbol BC549 -> Transistor_BJT:BC549
- R11: renamed from R2; footprint Resistors_THT:R_Axial_DIN0207_L6.3mm_D2.5mm_P10.16mm_Horizontal -> Resistor_THT:R_Axial_DIN0207_L6.3mm_D2.5mm_P10.16mm_Horizontal; symbol R -> Device:R
- R12: renamed from R3; footprint Resistors_THT:R_Axial_DIN0207_L6.3mm_D2.5mm_P10.16mm_Horizontal -> Resistor_THT:R_Axial_DIN0207_L6.3mm_D2.5mm_P10.16mm_Horizontal; symbol R -> Device:R
- R13: renamed from R7; footprint Resistors_THT:R_Axial_DIN0207_L6.3mm_D2.5mm_P10.16mm_Horizontal -> Resistor_THT:R_Axial_DIN0207_L6.3mm_D2.5mm_P10.16mm_Horizontal; symbol R -> Device:R
- R14: renamed from R12; footprint Resistors_THT:R_Axial_DIN0207_L6.3mm_D2.5mm_P10.16mm_Horizontal -> Resistor_THT:R_Axial_DIN0207_L6.3mm_D2.5mm_P10.16mm_Horizontal; symbol R -> Device:R
- R15: renamed from R4; footprint Resistors_THT:R_Axial_DIN0207_L6.3mm_D2.5mm_P10.16mm_Horizontal -> Resistor_THT:R_Axial_DIN0207_L6.3mm_D2.5mm_P10.16mm_Horizontal; symbol R -> Device:R
- R16: renamed from R5; footprint Resistors_THT:R_Axial_DIN0207_L6.3mm_D2.5mm_P10.16mm_Horizontal -> Resistor_THT:R_Axial_DIN0207_L6.3mm_D2.5mm_P10.16mm_Horizontal; symbol R -> Device:R
- R2: renamed from R6; footprint Resistors_THT:R_Axial_DIN0207_L6.3mm_D2.5mm_P10.16mm_Horizontal -> Resistor_THT:R_Axial_DIN0207_L6.3mm_D2.5mm_P10.16mm_Horizontal; symbol R -> Device:R
- R4: renamed from R1; footprint Resistors_THT:R_Axial_DIN0207_L6.3mm_D2.5mm_P10.16mm_Horizontal -> Resistor_THT:R_Axial_DIN0207_L6.3mm_D2.5mm_P10.16mm_Horizontal; symbol R -> Device:R
- R7: renamed from R8; footprint Resistors_THT:R_Axial_DIN0207_L6.3mm_D2.5mm_P10.16mm_Horizontal -> Resistor_THT:R_Axial_DIN0207_L6.3mm_D2.5mm_P10.16mm_Horizontal; symbol R -> Device:R
- R9: renamed from R11; footprint Resistors_THT:R_Axial_DIN0207_L6.3mm_D2.5mm_P10.16mm_Horizontal -> Resistor_THT:R_Axial_DIN0207_L6.3mm_D2.5mm_P10.16mm_Horizontal; symbol R -> Device:R
- U1: symbol LM7805_TO220 -> C64-Modulator-rescue:LM7805_TO220
Connections:
- wire segments 88 -> 138
Other:
- moved on the sheet: Q1, Q4

Commit message: Completed double-buffering Chroma/Luma split & library cleanup
Parts:
- removed J1, J2, J3, J4, J5, J6, J7, J8: (no value), anchors:anchor_circle, symbol C64-Modulator-rescue:Conn_01x01
- C5: renamed from C7; value 10uF -> 22uF
- C6: renamed from C8; value 100uF -> 10uF
- J1: renamed from J9; symbol 6569_modulator:6569_8765 -> Connector_Generic:Conn_01x04
- J2: renamed from J10; symbol 6569_modulator:6569_4321 -> Connector_Generic:Conn_01x04
- J3: renamed from J11; footprint Pin_Headers:Pin_Header_Straight_1x02_Pitch2.54mm -> Connector_PinHeader_2.54mm:PinHeader_1x02_P2.54mm_Vertical; symbol C64-Modulator-rescue:Conn_01x02 -> Connector_Generic:Conn_01x02
- J4: renamed from J12; symbol trs_3.5mm:TRS_3.5mm -> TRS-Plug:TRS_3.5mm
- J5: renamed from J13; symbol rca_plug:RCA_PLUG -> RCA-Plug:RCA_PLUG
- U1: footprint TO_SOT_Packages_THT:TO-220-3_Horizontal -> Package_TO_SOT_THT:TO-220-3_Horizontal_TabDown; symbol C64-Modulator-rescue:LM7805_TO220 -> Regulator_Linear:LM7805_TO220
- renumbered C4 to C1, C5 to C2, C6 to C4, C9 to C7, D2 to D1, D5 to D2, Q4 to Q1, Q3 to Q2, Q1 to Q3, Q2 to Q4, R4 to R1, R9 to R10, R13 to R11, R14 to R12, R11 to R2, R12 to R3, R2 to R4, R15 to R5, R8 to R6, R16 to R7, R7 to R8, R10 to R9
Other:
- note added: "Based on the C64 RF Modulator mod by Zero-X / OMS and suggested mods to the stock \nmodulator by Adrian’s Digital Basement. Chroma & Luma are separately buffered for the\nComposite & S-Video outputs to prevent interference."
- note added: "C64 Headers (250407)"
- note added: "Power Supply / Voltage Regulator"
- note removed: "Based on the C64 RF-modulator mod by Zero-X / OMS, this simply adapts those\nschematics with changes of my own to create a complete replacement for the\nmodulator. Given differences in pinouts this variant is meant for installation only on\nCommodore 64s with "longboards"."
- note removed: "C"
- note removed: "C64 Modulator replacement, "Longboard" edition"
- moved on the sheet: C1, C2, C5, C6, C7, D2, J1, J2, J3, J4, J5, JP1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

Commit message: Re-Add mounting point supports to main board (ground pins)
Parts:
- added J3, J4, J5, J6: Conn_01x01_Female, Connector_PinHeader_2.54mm:PinHeader_1x01_P2.54mm_Vertical, symbol Connector:Conn_01x01_Female
- J8: renamed from J4; symbol TRS-Plug:TRS_3.5mm -> trs_3.5mm:TRS_3.5mm
- J9: renamed from J5; symbol RCA-Plug:RCA_PLUG -> rca_plug:RCA_PLUG
- renumbered J3 to J7, R9 to R8, R8 to R9
Connections:
- net GND: now also J3.1 (Pin_1), J4.1 (Pin_1), J5.1 (Pin_1), J6.1 (Pin_1)
Other:
- note added: "Support attachments to\n main board."
Changed lines of the file:
@@
 	4725 6925 4725 7050
 $Comp
-L power:GND #PWR08
+L power:GND #PWR09
 U 1 1 5D0D1B71
 P 4725 7125
-F 0 "#PWR08" H 4725 6875 50  0001 C CNN
+F 0 "#PWR09" H 4725 6875 50  0001 C CNN
 F 1 "GND" H 4725 6975 50  0000 C CNN
 F 2 "" H 4725 7125 50  0001 C CNN
@@
 $EndComp
 $Comp
-L Device:R R8
+L Device:R R9
 U 1 1 5D0D23CC
 P 5100 6600
-F 0 "R8" V 5180 6600 50  0000 C CNN
+F 0 "R9" V 5180 6600 50  0000 C CNN
 F 1 "150" V 5100 6600 50  0000 C CNN
 F 2 "Resistor_THT:R_Axial_DIN0207_L6.3mm_D2.5mm_P10.16mm_Horizontal" V 5030 6600 50  0001 C CNN
@@
 	1050 7325 1050 7400
 $Comp
-L RCA-Plug:RCA_PLUG J5
+L rca_plug:RCA_PLUG J9
 U 1 1 5D0D8017
 P 9500 1150
-F 0 "J5" H 9510 1270 50  0000 C CNN
+F 0 "J9" H 9510 1270 50  0000 C CNN
 F 1 "RCA_PLUG" V 9615 1150 50  0000 C CNN
 F 2 "rca:rca_yellow" H 9500 1150 50  0001 C CNN
@@
 	9350 1150 9275 1150
 $Comp
-L power:GND #PWR015
+L power:GND #PWR016
 U 1 1 5D0D8DCE
 P 9650 1500
-F 0 "#PWR015" H 9650 1250 50  0001 C CNN
+F 0 "#PWR016" H 9650 1250 50  0001 C CNN
 F 1 "GND" H 9650 1350 50  0000 C CNN
 F 2 "" H 9650 1500 50  0001 C CNN
@@
 	9500 1350 9500 1425
 $Comp
-L TRS-Plug:TRS_3.5mm J4
+L trs_3.5mm:TRS_3.5mm J8
 U 1 1 5D0D92E8
 P 9300 1700
-F 0 "J4" H 9300 1990 50  0000 C CNN
+F 0 "J8" H 9300 1990 50  0000 C CNN
 F 1 "TRS_3.5mm" H 9150 1500 50  0000 L CNN
 F 2 "trs:Tayda_3.5mm_stereo_TRS_jack_A-853" H 9550 1800 50  0001 C CNN
@@
 	8475 2425 8350 2425
 $Comp
-L power:+9V #PWR03
+L power:+9V #PWR02
 U 1 1 5D4B6616
 P 2300 7150
-F 0 "#PWR03" H 2300 7000 50  0001 C CNN
+F 0 "#PWR02" H 2300 7000 50  0001 C CNN
 F 1 "+9V" H 2300 7290 50  0000 C CNN
 F 2 "" H 2300 7150 50  0001 C CNN
@@
 $EndComp
 $Comp
-L Connector_Generic:Conn_01x02 J3
+L Connector_Generic:Conn_01x02 J7
 U 1 1 5D55784F
 P 8150 2425
-F 0 "J3" H 8150 2525 50  0000 C CNN
+F 0 "J7" H 8150 2525 50  0000 C CNN
 F 1 "AUD_RIGHT" H 8150 2225 50  0000 C CNN
 F 2 "Connector_PinHeader_2.54mm:PinHeader_1x02_P2.54mm_Vertical" H 8150 2425 50  0001 C CNN
@@
 $EndComp
 $Comp
-L power:VCC #PWR07
+L power:VCC #PWR08
 U 1 1 5F74AF08
 P 4725 5675
-F 0 "#PWR07" H 4725 5525 50  0001 C CNN
+F 0 "#PWR08" H 4725 5525 50  0001 C CNN
 F 1 "VCC" H 4725 5825 50  0000 C CNN
 F 2 "" H 4725 5675 50  0001 C CNN
@@
 	4350 5975 4425 5975
 $Comp
-L power:GND #PWR010
+L power:GND #PWR012
 U 1 1 5F760EAB
 P 5950 5950
-F 0 "#PWR010" H 5950 5700 50  0001 C CNN
+F 0 "#PWR012" H 5950 5700 50  0001 C CNN
 F 1 "GND" H 5950 5800 50  0000 C CNN
 F 2 "" H 5950 5950 50  0001 C CNN
@@
 $EndComp
 $Comp
-L power:VCC #PWR06
+L power:VCC #PWR05
 U 1 1 5D0D18BE
 P 4550 4525
-F 0 "#PWR06" H 4550 4375 50  0001 C CNN
+F 0 "#PWR05" H 4550 4375 50  0001 C CNN
 F 1 "VCC" H 4550 4675 50  0000 C CNN
 F 2 "" H 4550 4525 50  0001 C CNN
@@
 	4725 5775 4725 5675
 $Comp
-L power:VCC #PWR04
+L power:VCC #PWR06
 U 1 1 5D0CC8F5
 P 4575 1275
-F 0 "#PWR04" H 4575 1125 50  0001 C CNN
+F 0 "#PWR06" H 4575 1125 50  0001 C CNN
 F 1 "VCC" H 4575 1425 50  0000 C CNN
 F 2 "" H 4575 1275 50  0001 C CNN
@@
 Connection ~ 2850 1950
 $Comp
-L power:GND #PWR02
+L power:GND #PWR04
 U 1 1 5D0CFC09
 P 2850 2750
-F 0 "#PWR02" H 2850 2500 50  0001 C CNN
+F 0 "#PWR04" H 2850 2500 50  0001 C CNN
 F 1 "GND" H 2850 2600 50  0000 C CNN
 F 2 "" H 2850 2750 50  0001 C CNN
@@
 	5025 4125 5025 4050
 $Comp
-L Device:R R9
+L Device:R R8
 U 1 1 5F7CE5BE
 P 5025 3900
-F 0 "R9" V 5105 3900 50  0000 C CNN
+F 0 "R8" V 5105 3900 50  0000 C CNN
 F 1 "220" V 5025 3900 50  0000 C CNN
 F 2 "Resistor_THT:R_Axial_DIN0207_L6.3mm_D2.5mm_P10.16mm_Horizontal" V 4955 3900 50  0001 C CNN
@@
 	4575 2950 4575 3200
 $Comp
-L power:VCC #PWR05
+L power:VCC #PWR07
 U 1 1 5F7CE580
 P 4575 2950
-F 0 "#PWR05" H 4575 2800 50  0001 C CNN
+F 0 "#PWR07" H 4575 2800 50  0001 C CNN
 F 1 "VCC" H 4575 3100 50  0000 C CNN
 F 2 "" H 4575 2950 50  0001 C CNN
@@
 $EndComp
 $Comp
-L power:GND #PWR09
+L power:GND #PWR011
 U 1 1 5F75C1CD
 P 5025 4125
-F 0 "#PWR09" H 5025 3875 50  0001 C CNN
+F 0 "#PWR011" H 5025 3875 50  0001 C CNN
 F 1 "GND" H 5025 3975 50  0000 C CNN
 F 2 "" H 5025 4125 50  0001 C CNN
@@
 	2050 1950 2850 1950
 $Comp
-L power:GND #PWR0101
+L power:GND #PWR010
 U 1 1 5F7B82A3
 P 5025 2675
-F 0 "#PWR0101" H 5025 2425 50  0001 C CNN
+F 0 "#PWR010" H 5025 2425 50  0001 C CNN
 F 1 "GND" H 5030 2502 50  0000 C CNN
 F 2 "" H 5025 2675 50  0001 C CNN
@@
 Connection ~ 10125 5875
 $Comp
-L power:VCC #PWR014
+L power:VCC #PWR017
 U 1 1 5D4BD9A3
 P 10125 5450
-F 0 "#PWR014" H 10125 5300 50  0001 C CNN
+F 0 "#PWR017" H 10125 5300 50  0001 C CNN
 F 1 "VCC" H 10125 5600 50  0000 C CNN
 F 2 "" H 10125 5450 50  0001 C CNN
@@
 $EndComp
 $Comp
-L power:GND #PWR012
+L power:GND #PWR015
 U 1 1 5D4BD167
 P 9350 6300
-F 0 "#PWR012" H 9350 6050 50  0001 C CNN
+F 0 "#PWR015" H 9350 6050 50  0001 C CNN
 F 1 "GND" H 9350 6150 50  0000 C CNN
 F 2 "" H 9350 6300 50  0001 C CNN
@@
 	9050 5875 8900 5875
 $Comp
-L power:+9V #PWR011
+L power:+9V #PWR014
 U 1 1 5D4BAC44
 P 8900 5725
-F 0 "#PWR011" H 8900 5575 50  0001 C CNN
+F 0 "#PWR014" H 8900 5575 50  0001 C CNN
 F 1 "+9V" H 8900 5865 50  0000 C CNN
 F 2 "" H 8900 5725 50  0001 C CNN
@@
 	1    0    0    -1
 $EndComp
+$Comp
+L Connector:Conn_01x01_Female J3
+U 1 1 5F7D23BF
+P 2975 6425
+F 0 "J3" H 3003 6451 50  0000 L CNN
+F 1 "Conn_01x01_Female" H 3003 6360 50  0000 L CNN
+F 2 "Connector_PinHeader_2.54mm:PinHeader_1x01_P2.54mm_Vertical" H 2975 6425 50  0001 C CNN
+F 3 "~" H 2975 6425 50  0001 C CNN
+	1    2975 6425
+	1    0    0    -1
+$EndComp
+$Comp
+L Connector:Conn_01x01_Female J4
+U 1 1 5F7D2B72
+P 2975 6625
+F 0 "J4" H 3003 6651 50  0000 L CNN
+F 1 "Conn_01x01_Female" H 3003 6560 50  0000 L CNN
+F 2 "Connector_PinHeader_2.54mm:PinHeader_1x01_P2.54mm_Vertical" H 2975 6625 50  0001 C CNN
+F 3 "~" H 2975 6625 50  0001 C CNN
+	1    2975 6625
+	1    0    0    -1
+$EndComp
+$Comp
+L Connector:Conn_01x01_Female J5
+U 1 1 5F7D3860
+P 2975 6875
+F 0 "J5" H 3003 6901 50  0000 L CNN
+F 1 "Conn_01x01_Female" H 3003 6810 50  0000 L CNN
+F 2 "Connector_PinHeader_2.54mm:PinHeader_1x01_P2.54mm_Vertical" H 2975 6875 50  0001 C CNN
+F 3 "~" H 2975 6875 50  0001 C CNN
+	1    2975 6875
+	1    0    0    -1
+$EndComp
+$Comp
+L Connector:Conn_01x01_Female J6
+U 1 1 5F7D4447
+P 2975 7075
+F 0 "J6" H 3003 7101 50  0000 L CNN
+F 1 "Conn_01x01_Female" H 3003 7010 50  0000 L CNN
+F 2 "Connector_PinHeader_2.54mm:PinHeader_1x01_P2.54mm_Vertical" H 2975 7075 50  0001 C CNN
+F 3 "~" H 2975 7075 50  0001 C CNN
+	1    2975 7075
+	1    0    0    -1
+$EndComp
+$Comp
+L power:GND #PWR03
+U 1 1 5F7D5BDA
+P 2775 7150
+F 0 "#PWR03" H 2775 6900 50  0001 C CNN
+F 1 "GND" H 2780 6977 50  0000 C CNN
+F 2 "" H 2775 7150 50  0001 C CNN
+F 3 "" H 2775 7150 50  0001 C CNN
+	1    2775 7150
+	1    0    0    -1
+$EndComp
+Wire Wire Line
+	2775 6425 2775 6625
+Connection ~ 2775 6625
+Wire Wire Line
+	2775 6625 2775 6875
+Connection ~ 2775 6875
+Wire Wire Line
+	2775 6875 2775 7075
+Connection ~ 2775 7075
+Wire Wire Line
+	2775 7075 2775 7150
+Wire Notes Line
+	2600 6250 4150 6250
+Wire Notes Line
+	4150 6250 4150 7925
+Wire Notes Line
+	4150 7925 2600 7925
+Wire Notes Line
+	2600 7925 2600 6250
+Text Notes 2775 7875 0    60   ~ 0
+Support attachments to\n     main board.
 $EndSCHEMATC

Commit message: Add mounting supports under RCA & TRS jack.
Parts:
- added J10, J11: Conn_01x01_Female, Connector_PinHeader_2.54mm:PinHeader_1x01_P2.54mm_Vertical, symbol Connector:Conn_01x01_Female
- J8: symbol trs_3.5mm:TRS_3.5mm -> TRS_Jack:TRS_3.5mm
- J9: symbol rca_plug:RCA_PLUG -> RCA_Jack:RCA_PLUG
Connections:
- net GND: now also J10.1 (Pin_1), J11.1 (Pin_1)
Changed lines of the file:
@@
 	1050 7325 1050 7400
 $Comp
-L rca_plug:RCA_PLUG J9
+L RCA_Jack:RCA_PLUG J9
 U 1 1 5D0D8017
 P 9500 1150
@@
 	9500 1350 9500 1425
 $Comp
-L trs_3.5mm:TRS_3.5mm J8
+L TRS_Jack:TRS_3.5mm J8
 U 1 1 5D0D92E8
 P 9300 1700
@@
 L power:GND #PWR03
 U 1 1 5F7D5BDA
-P 2775 7150
-F 0 "#PWR03" H 2775 6900 50  0001 C CNN
-F 1 "GND" H 2780 6977 50  0000 C CNN
-F 2 "" H 2775 7150 50  0001 C CNN
-F 3 "" H 2775 7150 50  0001 C CNN
-	1    2775 7150
+P 2775 7525
+F 0 "#PWR03" H 2775 7275 50  0001 C CNN
+F 1 "GND" H 2780 7352 50  0000 C CNN
+F 2 "" H 2775 7525 50  0001 C CNN
+F 3 "" H 2775 7525 50  0001 C CNN
+	1    2775 7525
 	1    0    0    -1
 $EndComp
@@
 Wire Wire Line
 	2775 6875 2775 7075
-Connection ~ 2775 7075
-Wire Wire Line
-	2775 7075 2775 7150
 Wire Notes Line
 	2600 6250 4150 6250
@@
 Text Notes 2775 7875 0    60   ~ 0
 Support attachments to\n     main board.
+$Comp
+L Connector:Conn_01x01_Female J10
+U 1 1 6048DE81
+P 2975 7250
+F 0 "J10" H 3003 7276 50  0000 L CNN
+F 1 "Conn_01x01_Female" H 3003 7185 50  0000 L CNN
+F 2 "Connector_PinHeader_2.54mm:PinHeader_1x01_P2.54mm_Vertical" H 2975 7250 50  0001 C CNN
+F 3 "~" H 2975 7250 50  0001 C CNN
+	1    2975 7250
+	1    0    0    -1
+$EndComp
+$Comp
+L Connector:Conn_01x01_Female J11
+U 1 1 604928C9
+P 2975 7425
+F 0 "J11" H 3003 7451 50  0000 L CNN
+F 1 "Conn_01x01_Female" H 3003 7360 50  0000 L CNN
+F 2 "Connector_PinHeader_2.54mm:PinHeader_1x01_P2.54mm_Vertical" H 2975 7425 50  0001 C CNN
+F 3 "~" H 2975 7425 50  0001 C CNN
+	1    2975 7425
+	1    0    0    -1
+$EndComp
+Wire Wire Line
+	2775 7075 2775 7250
+Connection ~ 2775 7075
+Wire Wire Line
+	2775 7250 2775 7425
+Connection ~ 2775 7250
+Wire Wire Line
+	2775 7425 2775 7525
+Connection ~ 2775 7425
 $EndSCHEMATC
